Commit message: configuration opérationnelle

File: sc_tutorial_description/config/sc_tutorial.config.xacro (robot description, xacro)
@@ -1,12 +1,6 @@
 <?xml version="1.0"?>
-<!-- Scara manipulator -->
-<robot xmlns:xacro="http://www.ros.org/wiki/xacro" name="scara">
-    <!-- Import scara urdf file -->
-    <xacro:include filename="$(find scara_description)/urdf/scara.urdf" />
-    <!-- Import scara materials file -->
-    <xacro:include filename="$(find scara_description)/config/materials.urdf" />
-    <!-- Import scara ros2_control description -->
-    <xacro:include filename="$(find scara_description)/ros2_control/scara.ros2_control.urdf" />
-    <!-- Import all Gazebo-customization elements -->
-    <xacro:include filename="$(find scara_description)/gazebo/scara.gazebo.xacro"/>
+<robot xmlns:xacro="http://www.ros.org/wiki/xacro" name="motor_drive">
+  <link name="world"/>
+  <xacro:include filename="$(find sc_tutorial_description)/ros2_control/sc_tutorial.ros2_control.xacro" />
+  <xacro:motor_drive/>
 </robot>

File: sc_tutorial_description/ros2_control/sc_tutorial.ros2_control.xacro (robot description, xacro)
@@ -10,8 +10,13 @@
    <gpio name="gpio_0">
       <state_interface name="status"/>
-      <state_interface name="position"/>
+      <state_interface name="value"/>
       <command_interface name="ctrl"/>
       <command_interface name="position"/>
       <command_interface name="latch_value"/>
+      <command_interface name="status"/>
+      <command_interface name="value"/>
+      <state_interface name="ctrl"/>
+      <state_interface name="position"/>
+      <state_interface name="latch_value"/>
       <ec_module name="EL5101">
         <plugin>ethercat_generic_plugins/GenericEcSlave</plugin>
@@ -24,4 +29,6 @@
       <command_interface name="analog_output.1"/>
       <command_interface name="analog_output.2"/>
+      <state_interface name="analog_output.1"/>
+      <state_interface name="analog_output.2"/>
       <ec_module name="EL4132">
         <plugin>ethercat_generic_plugins/GenericEcSlave</plugin>
@@ -34,4 +41,6 @@
       <state_interface name="analog_input.1"/>
       <state_interface name="analog_input.2"/>
+      <command_interface name="analog_input.1"/>
+      <command_interface name="analog_input.2"/>
       <ec_module name="EL3102">
         <plugin>ethercat_generic_plugins/GenericEcSlave</plugin>
